File: root.brd (EAGLE design)
At the start: 100 x 87 mm, 34 parts, among them X1 MKDSN1,5/3-5,08, X2 MKDSN1,5/2-5,08, X3 MKDSN1,5/2-5,08, X4 MKDSN1,5/2-5,08, X5 MKDSN1,5/2-5,08, X6 MKDSN1,5/2-5,08, X7 MKDSN1,5/2-5,08, X8 MKDSN1,5/2-5,08, X9 MKDSN1,5/2-5,08

Commit message: released
Parts:
- R7, R9: value 1k 1W -> 1k 0.1W
Changed lines of the file:
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@@
 <element name="R6" library="rcl" package="R2512" value="22k 1W" x="54.5" y="13.5" rot="R90"/>
 <element name="C4" library="resistor" package="PANASONIC_F" value="100uF 100V" x="47.5" y="17.5" rot="R270"/>
-<element name="R7" library="resistor" package="R0603" value="1k 1W" x="41.5" y="17.5" rot="R270"/>
+<element name="R7" library="resistor" package="R0603" value="1k 0.1W" x="41.5" y="17.5" rot="R270"/>
 <element name="R8" library="rcl" package="R2512" value="10k 1W" x="35.5" y="18" rot="R90"/>
 <element name="C2" library="resistor" package="PANASONIC_F" value="100uF 100V" x="28" y="17.5" rot="R270"/>
-<element name="R9" library="resistor" package="R0603" value="1k 1W" x="39.5" y="17.5" rot="R90"/>
+<element name="R9" library="resistor" package="R0603" value="1k 0.1W" x="39.5" y="17.5" rot="R90"/>
 </elements>
 <signals>
