File: root.sch (EAGLE design)
At the start: 34 parts, among them X1 MKDSN1,5/3-5,08, X2 MKDSN1,5/2-5,08, X3 MKDSN1,5/2-5,08, X4 MKDSN1,5/2-5,08, X5 MKDSN1,5/2-5,08, X6 MKDSN1,5/2-5,08, X7 MKDSN1,5/2-5,08, X8 MKDSN1,5/2-5,08, X9 MKDSN1,5/2-5,08

Commit message: released
Parts:
- R7, R9: value 1k 1W -> 1k 0.1W
Changed lines of the file:
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@@
 <part name="R6" library="rcl" deviceset="R-EU_" device="R2512" value="22k 1W"/>
 <part name="C4" library="resistor" deviceset="CPOL-US" device="F" value="100uF 100V"/>
-<part name="R7" library="resistor" deviceset="R-EU_" device="R0603" value="1k 1W"/>
+<part name="R7" library="resistor" deviceset="R-EU_" device="R0603" value="1k 0.1W"/>
 <part name="R8" library="rcl" deviceset="R-EU_" device="R2512" value="10k 1W"/>
 <part name="C2" library="resistor" deviceset="CPOL-US" device="F" value="100uF 100V"/>
-<part name="R9" library="resistor" deviceset="R-EU_" device="R0603" value="1k 1W"/>
+<part name="R9" library="resistor" deviceset="R-EU_" device="R0603" value="1k 0.1W"/>
 </parts>
 <sheets>
